Commit message: Update sensor configuration

File: rbcar_description/robots/rbcar.urdf.xacro (robot description, xacro)
@@ -1,5 +1,5 @@
 <?xml version="1.0"?>
-  <robot name="rbcar"
-    xmlns:xacro="http://wiki.ros.org/xacro">
+<robot name="rbcar"
+	xmlns:xacro="http://wiki.ros.org/xacro">
 	<!-- ***************** -->
 	<!-- Imported elements -->
@@ -10,5 +10,5 @@
 	<!-- Import Robotnik CAR wheels -->
 	<xacro:include filename="$(find rbcar_description)/urdf/wheels/suspension_wheel_v2.urdf.xacro" />
-	<xacro:include filename="$(find rbcar_description)/urdf/structures/elevator.urdf.xacro" />
+	<!-- <xacro:include filename="$(find rbcar_description)/urdf/structures/elevator.urdf.xacro" /> -->
 	<!-- Import all available sensors -->
 	<xacro:include filename="$(find robotnik_sensors)/urdf/all_sensors.urdf.xacro" />
@@ -18,5 +18,6 @@
 	<xacro:property name="PI" value="3.1415926535897931"/>
 	<!-- Wheel parameters -->
-	<xacro:property name="wheel_offset_x" value="1.0" />    <!-- x,y,z in translation from base_link to the center of the wheel -->
+	<xacro:property name="wheel_offset_x" value="1.0" />
+	<!-- x,y,z in translation from base_link to the center of the wheel -->
 	<xacro:property name="wheel_offset_y" value="0.75" />
 	<xacro:property name="wheel_offset_z" value="0.0" />
@@ -31,43 +32,28 @@
 	<!-- Gazebo ros control pluggins -->
 	<xacro:ros_control/>
-        <!-- xacro:omni_steering prefix="" publish_tf="true"/-->
+	<!-- xacro:omni_steering prefix="" publish_tf="true"/-->
 	<!-- Gazebo skid steering pluggins -->
 	<!-- xacro:skid_steering broadcastOdomTF="1"/ -->
 	<!-- WHEELS -->
-    <!-- Wheels -->
-    <xacro:front_wheel lr_prefix="left" fr_prefix="front"
-                       lr_reflect="1" fr_reflect="1" parent="base_link" />
-    <xacro:front_wheel lr_prefix="right" fr_prefix="front"
-                       lr_reflect="-1" fr_reflect="1" parent="base_link" />
-    <xacro:rear_wheel lr_prefix="left" fr_prefix="rear"
-                      lr_reflect="1" fr_reflect="-1" parent="base_link" />
-    <xacro:rear_wheel lr_prefix="right" fr_prefix="rear"
-                      lr_reflect="-1" fr_reflect="-1" parent="base_link" />
+	<!-- Wheels -->
+	<xacro:front_wheel lr_prefix="left" fr_prefix="front" lr_reflect="1" fr_reflect="1" parent="base_link" />
+	<xacro:front_wheel lr_prefix="right" fr_prefix="front" lr_reflect="-1" fr_reflect="1" parent="base_link" />
+	<xacro:rear_wheel lr_prefix="left" fr_prefix="rear" lr_reflect="1" fr_reflect="-1" parent="base_link" />
+	<xacro:rear_wheel lr_prefix="right" fr_prefix="rear" lr_reflect="-1" fr_reflect="-1" parent="base_link" />
 	<!-- SENSORS -->
-  <!--xacro:sensor_benewake_ce30d prefix="front_3d_lidar" parent="base_link" gpu="true">
-      <origin xyz="2.155 0.0 0.236" rpy="0 0.24396 0"/>
-  </xacro:sensor_benewake_ce30d-->
-  <xacro:sensor_velodyne_vlp16 prefix="front_3d_lidar" parent="base_link" range_min="0.8" range_max="31.0" gpu="false">
-      <origin xyz="2.155 0.0 0.236" rpy="0 0.24396 0"/>
-  </xacro:sensor_velodyne_vlp16>
-  <xacro:sensor_rubedos_viper prefix="viper" parent="base_link">
-    <origin xyz="1.289 0.0 1.354" rpy="0 0.1745 0.0"/>
-  </xacro:sensor_rubedos_viper>
+	<xacro:sensor_velodyne_vlp16 prefix="front_3d_lidar" parent="base_link" range_min="0.8" range_max="31.0" gpu="false">
+		<origin xyz="1.19 0.0 1.54" rpy="0 0.24396 0"/>
+	</xacro:sensor_velodyne_vlp16>
+	<xacro:sensor_rubedos_viper prefix="viper" parent="base_link">
+		<origin xyz="1.58 0.0 0.87" rpy="0 0 0.0"/>
+	</xacro:sensor_rubedos_viper>
 	<xacro:sensor_imu_hector prefix="imu" parent="base_link">
 		<origin xyz="0.0 0.0 0.170" rpy="0 0 0"/>
-		<!--<origin xyz="0.917 0.0 0.170" rpy="0 0 0"/>-->
 	</xacro:sensor_imu_hector>
-  <!--xacro:sensor_sick_s300 prefix="front_laser" parent="base_link" prefix_topic="front_laser" min_angle="-1.5" max_angle="1.5" gpu="false">
-    <origin xyz="2.2 0 0.3" rpy="0 0 0"/>
-  </xacro:sensor_sick_s300-->
+	<xacro:sensor_sick_s300 prefix="front_laser" parent="base_link" prefix_topic="front_laser" min_angle="-1.5" max_angle="1.5" gpu="false">
+		<origin xyz="2.2 0 0.3" rpy="0 0 0"/>
+	</xacro:sensor_sick_s300>
 	<xacro:sensor_gps prefix="gps" parent="base_link" gps_latitude="$(arg gps_latitude)" gps_longitude="$(arg gps_longitude)">
-		<origin xyz="0.0 0 1.5" rpy="0 0 0"/>
-		<!--<origin xyz="0.747 0 1.5" rpy="0 0 0"/>-->
+		<origin xyz="0.0 0 0.45" rpy="0 0 0"/>
 	</xacro:sensor_gps>
-  <xacro:elevator parent="base_link">
-		<origin xyz="0.0 0.0 0.6" rpy="0 0 0"/>
-	</xacro:elevator>
-  <xacro:sensor_axis prefix="front_ptz_camera" parent="elevator_link">
-    <origin xyz="0 0 0" rpy="0 0 0"/>
-  </xacro:sensor_axis>
 </robot>

Commit message: Update Velodyne sensor

File: rbcar_description/robots/rbcar.urdf.xacro (robot description, xacro)
@@ -13,4 +13,5 @@
 	<!-- Import all available sensors -->
 	<xacro:include filename="$(find robotnik_sensors)/urdf/all_sensors.urdf.xacro" />
+	<xacro:include filename="$(find velodyne_description)/urdf/VLP-16.urdf.xacro"/>
 	<!-- ***************** -->
 	<!-- Global parameters -->
@@ -42,7 +43,11 @@
 	<xacro:rear_wheel lr_prefix="right" fr_prefix="rear" lr_reflect="-1" fr_reflect="-1" parent="base_link" />
 	<!-- SENSORS -->
+	<!--
 	<xacro:sensor_velodyne_vlp16 prefix="front_3d_lidar" parent="base_link" range_min="0.8" range_max="31.0" gpu="false">
 		<origin xyz="1.19 0.0 1.54" rpy="0 0.24396 0"/>
-	</xacro:sensor_velodyne_vlp16>
+	</xacro:sensor_velodyne_vlp16> -->
+	<VLP-16 parent="base_link" name="velodyne" topic="/velodyne_points" hz="10" samples="440" min_range="0.9" max_range="100.0" gpu="false">
+		<origin xyz="1.19 0.0 1.54" rpy="0 0.24396 0" /> <!-- 13.97787837 deg -->
+	</VLP-16>
 	<xacro:sensor_rubedos_viper prefix="viper" parent="base_link">
 		<origin xyz="1.58 0.0 0.87" rpy="0 0 0.0"/>

Commit message: Add ground truth plugin and fix controller

File: rbcar_description/robots/rbcar.urdf.xacro (robot description, xacro)
@@ -42,4 +42,17 @@
 	<xacro:rear_wheel lr_prefix="left" fr_prefix="rear" lr_reflect="1" fr_reflect="-1" parent="base_link" />
 	<xacro:rear_wheel lr_prefix="right" fr_prefix="rear" lr_reflect="-1" fr_reflect="-1" parent="base_link" />
+	<!-- Ground truth plugin -->
+	<gazebo>
+		<plugin name="p3d_base_controller" filename="libgazebo_ros_p3d.so">
+			<alwaysOn>true</alwaysOn>
+			<updateRate>50.0</updateRate>
+			<bodyName>base_link</bodyName>
+			<topicName>ground_truth/state</topicName>
+			<gaussianNoise>0.01</gaussianNoise>
+			<frameName>map</frameName>
+			<xyzOffsets>0 0 0</xyzOffsets>
+			<rpyOffsets>0 0 0</rpyOffsets>
+		</plugin>
+	</gazebo>
 	<!-- SENSORS -->
 	<!--
@@ -48,5 +61,6 @@
 	</xacro:sensor_velodyne_vlp16> -->
 	<VLP-16 parent="base_link" name="velodyne" topic="/velodyne_points" hz="10" samples="440" min_range="0.9" max_range="100.0" gpu="false">
-		<origin xyz="1.19 0.0 1.54" rpy="0 0.24396 0" /> <!-- 13.97787837 deg -->
+		<origin xyz="1.19 0.0 1.55" rpy="0 0.24396 0" />
+		<!-- 13.97787837 deg -->
 	</VLP-16>
 	<xacro:sensor_rubedos_viper prefix="viper" parent="base_link">

Commit message: Modify navigation parameters

File: rbcar_description/robots/rbcar.urdf.xacro (robot description, xacro)
@@ -60,6 +60,6 @@
 		<origin xyz="1.19 0.0 1.54" rpy="0 0.24396 0"/>
 	</xacro:sensor_velodyne_vlp16> -->
-	<VLP-16 parent="base_link" name="velodyne" topic="/velodyne_points" hz="10" samples="440" min_range="0.9" max_range="100.0" gpu="false">
-		<origin xyz="1.19 0.0 1.55" rpy="0 0.24396 0" />
+	<VLP-16 parent="base_link" name="velodyne" topic="/velodyne_points" hz="10" samples="440" min_range="0.9" max_range="100.0" gpu="true">
+		<origin xyz="1.19 0.0 1.55" rpy="0 0.24396 0" /> <!-- 0.24396 -->
 		<!-- 13.97787837 deg -->
 	</VLP-16>
@@ -70,7 +70,7 @@
 		<origin xyz="0.0 0.0 0.170" rpy="0 0 0"/>
 	</xacro:sensor_imu_hector>
-	<xacro:sensor_sick_s300 prefix="front_laser" parent="base_link" prefix_topic="front_laser" min_angle="-1.5" max_angle="1.5" gpu="false">
+	<xacro:sensor_sick_microscan3 prefix="front_laser" parent="base_link" prefix_topic="front_laser" max_angle="2.3562" min_angle="-2.3562">
 		<origin xyz="2.2 0 0.3" rpy="0 0 0"/>
-	</xacro:sensor_sick_s300>
+	</xacro:sensor_sick_microscan3>
 	<xacro:sensor_gps prefix="gps" parent="base_link" gps_latitude="$(arg gps_latitude)" gps_longitude="$(arg gps_longitude)">
 		<origin xyz="0.0 0 0.45" rpy="0 0 0"/>

Commit message: Update sensor configuration

File: rbcar_description/robots/rbcar.urdf.xacro (robot description, xacro)
@@ -61,18 +61,26 @@
 	</xacro:sensor_velodyne_vlp16> -->
 	<VLP-16 parent="base_link" name="velodyne" topic="/velodyne_points" hz="10" samples="440" min_range="0.9" max_range="100.0" gpu="true">
-		<origin xyz="1.19 0.0 1.55" rpy="0 0.24396 0" /> <!-- 0.24396 -->
-		<!-- 13.97787837 deg -->
+		<origin xyz="1.19 0.0 1.55" rpy="0 0.24396 0" />
+		<!-- 0.24396 == 13.97787837 deg -->
 	</VLP-16>
-	<xacro:sensor_rubedos_viper prefix="viper" parent="base_link">
+	<!-- Front -->
+	<xacro:sensor_rubedos_viper prefix="front_viper" parent="base_link">
 		<origin xyz="1.58 0.0 0.87" rpy="0 0 0.0"/>
 	</xacro:sensor_rubedos_viper>
+	<xacro:sensor_sick_microscan3 prefix="front_laser" parent="base_link" prefix_topic="front_laser" max_angle="1.5708" min_angle="-1.5708">		<!-- initial angle value was : 2.3562 -->
+		<origin xyz="2.2 0 0.3" rpy="0 0 0"/>
+	</xacro:sensor_sick_microscan3>
+	<!-- Rear -->
+	<xacro:sensor_rubedos_viper prefix="rear_viper" parent="base_link">
+		<origin xyz="-0.15 0.0 0.475" rpy="0 0 3.14159"/>
+	</xacro:sensor_rubedos_viper>
+	<xacro:sensor_sick_microscan3 prefix="rear_laser" parent="base_link" prefix_topic="rear_laser" max_angle="1.309" min_angle="-1.309">
+		<origin xyz="-0.24 0 0.00" rpy="0 0 3.14159"/>
+	</xacro:sensor_sick_microscan3> <!-- 150 degrees -->
 	<xacro:sensor_imu_hector prefix="imu" parent="base_link">
 		<origin xyz="0.0 0.0 0.170" rpy="0 0 0"/>
 	</xacro:sensor_imu_hector>
-	<xacro:sensor_sick_microscan3 prefix="front_laser" parent="base_link" prefix_topic="front_laser" max_angle="1.5708" min_angle="-1.5708"> <!-- initial angle value was : 2.3562 . Changing it to 180 degrees to remove noise from RBCAR body -->
-		<origin xyz="2.2 0 0.3" rpy="0 0 0"/>
-	</xacro:sensor_sick_microscan3>
-	<xacro:sensor_gps prefix="gps" parent="base_link" gps_latitude="$(arg gps_latitude)" gps_longitude="$(arg gps_longitude)">
+	<!-- <xacro:sensor_gps prefix="gps" parent="base_link" gps_latitude="$(arg gps_latitude)" gps_longitude="$(arg gps_longitude)">
 		<origin xyz="0.0 0 0.45" rpy="0 0 0"/>
-	</xacro:sensor_gps>
+	</xacro:sensor_gps> -->
 </robot>

Commit message: Update parameters

File: rbcar_description/robots/rbcar.urdf.xacro (robot description, xacro)
@@ -42,5 +42,5 @@
 	<xacro:rear_wheel lr_prefix="left" fr_prefix="rear" lr_reflect="1" fr_reflect="-1" parent="base_link" />
 	<xacro:rear_wheel lr_prefix="right" fr_prefix="rear" lr_reflect="-1" fr_reflect="-1" parent="base_link" />
-	<!-- Ground truth plugin -->
+	<!-- Ground truth plugin-->
 	<gazebo>
 		<plugin name="p3d_base_controller" filename="libgazebo_ros_p3d.so">
@@ -56,9 +56,5 @@
 	</gazebo>
 	<!-- SENSORS -->
-	<!--
-	<xacro:sensor_velodyne_vlp16 prefix="front_3d_lidar" parent="base_link" range_min="0.8" range_max="31.0" gpu="false">
-		<origin xyz="1.19 0.0 1.54" rpy="0 0.24396 0"/>
-	</xacro:sensor_velodyne_vlp16> -->
-	<VLP-16 parent="base_link" name="velodyne" topic="/velodyne_points" hz="10" samples="440" min_range="0.9" max_range="100.0" gpu="true">
+	<VLP-16 parent="base_link" name="velodyne" topic="/points_raw" hz="10" samples="440" min_range="0.9" max_range="100.0" gpu="true">
 		<origin xyz="1.19 0.0 1.55" rpy="0 0.24396 0" />
 		<!-- 0.24396 == 13.97787837 deg -->
@@ -73,5 +69,6 @@
 	<!-- Rear -->
 	<xacro:sensor_rubedos_viper prefix="rear_viper" parent="base_link">
-		<origin xyz="-0.15 0.0 0.475" rpy="0 0 3.14159"/>
+		<origin xyz="0.42 0.0 1.55" rpy="0 0.24396 3.14159"/>
+		<!-- <origin xyz="-0.15 0.0 0.475" rpy="0 0 3.14159"/> -->
 	</xacro:sensor_rubedos_viper>
 	<xacro:sensor_sick_microscan3 prefix="rear_laser" parent="base_link" prefix_topic="rear_laser" max_angle="1.309" min_angle="-1.309">

Commit message: Update robot model to real specs

File: rbcar_description/robots/rbcar.urdf.xacro (robot description, xacro)
@@ -13,5 +13,4 @@
 	<!-- Import all available sensors -->
 	<xacro:include filename="$(find robotnik_sensors)/urdf/all_sensors.urdf.xacro" />
-	<xacro:include filename="$(find velodyne_description)/urdf/VLP-16.urdf.xacro"/>
 	<!-- ***************** -->
 	<!-- Global parameters -->
@@ -47,39 +46,4 @@
 	  <origin xyz="0 0.0 0" rpy="1.57079633 0 3.14159265"/>
     </xacro:rear_axle>
-	<!-- Ground truth plugin-->
-	<gazebo>
-		<plugin name="p3d_base_controller" filename="libgazebo_ros_p3d.so">
-			<alwaysOn>true</alwaysOn>
-			<updateRate>50.0</updateRate>
-			<bodyName>base_link</bodyName>
-			<topicName>ground_truth/state</topicName>
-			<gaussianNoise>0.01</gaussianNoise>
-			<frameName>map</frameName>
-			<xyzOffsets>0 0 0</xyzOffsets>
-			<rpyOffsets>0 0 0</rpyOffsets>
-		</plugin>
-	</gazebo>
-	<!-- SENSORS -->
-	<VLP-16 parent="base_link" name="velodyne" topic="/points_raw" hz="10" samples="440" min_range="0.9" max_range="100.0" gpu="true">
-		<origin xyz="1.19 0.0 1.55" rpy="0 0.24396 0" />
-		<!-- 0.24396 == 13.97787837 deg -->
-	</VLP-16>
-	<!-- Front -->
-	<xacro:sensor_rubedos_viper prefix="front_viper" parent="base_link">
-		<origin xyz="1.58 0.0 0.87" rpy="0 0 0.0"/>
-	</xacro:sensor_rubedos_viper>
-	<xacro:sensor_sick_microscan3 prefix="front_laser" parent="base_link" prefix_topic="front_laser" max_angle="1.5708" min_angle="-1.5708">		<!-- initial angle value was : 2.3562 -->
-		<origin xyz="2.2 0 0.3" rpy="0 0 0"/>
-	</xacro:sensor_sick_microscan3>
-	<!-- Rear -->
-	<xacro:sensor_rubedos_viper prefix="rear_viper" parent="base_link">
-		<origin xyz="0.42 0.0 1.55" rpy="0 0.24396 3.14159"/>
-		<!-- <origin xyz="-0.15 0.0 0.475" rpy="0 0 3.14159"/> -->
-  </xacro:sensor_rubedos_viper>
-	<xacro:sensor_sick_microscan3 prefix="rear_laser" parent="base_link" prefix_topic="rear_laser" max_angle="1.309" min_angle="-1.309">
-		<origin xyz="-0.24 0 0.00" rpy="0 0 3.14159"/>
-	</xacro:sensor_sick_microscan3> <!-- 150 degrees -->
-	<xacro:sensor_imu_hector prefix="imu" parent="base_link">
-		<origin xyz="0.0 0.0 0.170" rpy="0 0 0"/>
 	<xacro:sensor_rslidar_16 prefix="$(arg prefix)top_3d_laser" parent="$(arg prefix)base_link">
 	  <origin xyz="1.163 0.0 1.602" rpy="0 0.2637 0"/>
